File: bigMacro.kicad_sch (KiCad schematic)
At the start: 0 parts

Commit message: Initial PCB Design (Unfinished)
Started work on the keyboard layout
Parts:
- added D1, D2: SK6812MINI, LED_SMD:LED_SK6812MINI_PLCC4_3.5x3.5mm_P1.75mm, symbol LED:SK6812MINI
- added R1, R3: 22, symbol Device:R_Small
- added R2: 10k, symbol Device:R_Small
- added U1: ATmega32U4-A, Package_QFP:TQFP-44_10x10mm_P0.8mm, symbol MCU_Microchip_ATmega:ATmega32U4-A
Connections:
- new net: R3.2, U1.3 (D-)
- new net: R2.1, U1.33 (~{HWB}/PE2)
- new net: R1.2, U1.4 (D+)
- new net +5V: U1.14 (VCC), U1.2 (UVCC), U1.24 (AVCC), U1.34 (VCC), U1.44 (AVCC)
- new net GND: R2.2, U1.15 (GND), U1.23 (GND), U1.35 (GND), U1.43 (GND), U1.5 (UGND)

Commit message: Finished Base PCB Layout
Parts:
- removed D1, D2: SK6812MINI, LED_SMD:LED_SK6812MINI_PLCC4_3.5x3.5mm_P1.75mm, symbol LED:SK6812MINI
- added C1: 1uF, Capacitor_SMD:C_0805_2012Metric, symbol Device:C_Small
- added C2, C3, C4, C5: 0.1uF, Capacitor_SMD:C_0805_2012Metric, symbol Device:C_Small
- added C6, C7: 22pF, Capacitor_SMD:C_0805_2012Metric, symbol Device:C_Small
- added D1, D2, D3, D4: D_Small, Diode_SMD:D_SOD-123, symbol Device:D_Small
- added F1: Polyfuse_Small, Fuse:Fuse_1206_3216Metric, symbol Device:Polyfuse_Small
- added MX1, MX2, MX3, MX4: MX-NoLED, Button_Switch_Keyboard:SW_Cherry_MX_1.00u_PCB, symbol MXAH:MX-NoLED
- added R4: 10k, Resistor_SMD:R_0805_2012Metric, symbol Device:R_Small
- added SW1: SW_Push, Button_Switch_Keyboard:SW_Cherry_MX_1.00u_PCB, symbol Switch:SW_Push
- added USB1: Molex-0548190589, PRAND:Molex-0548190589, symbol PRAND:Molex-0548190589
- added Y1: 16MHz, Crystal:Crystal_SMD_3225-4Pin_3.2x2.5mm, symbol Device:Crystal_GND24_Small
- R1, R2, R3: footprint (none) -> Resistor_SMD:R_0805_2012Metric
Connections:
- net +5V: now also U1.7 (VBUS), C2.1, C3.1, C4.1, C5.1, F1.2, R4.1
- net GND: now also C1.2, C2.2, C3.2, C4.2, C5.2, C6.1, C7.1, SW1.1, USB1.1 (GND), Y1.1, Y1.3
- net D-: now reaches R3.1
- net D-: now also USB1.4 (D-)
- net at U1.13 (~{RESET}): now also R4.2, SW1.2
- net at U1.16 (XTAL2): now also C7.2, Y1.2
- net at U1.17 (XTAL1): now also C6.2, Y1.4
- net at U1.6 (UCAP): now also C1.1
- net D+: now reaches R1.1
- net D+: now also USB1.3 (D+)
- new net: D4.2 (A), MX4.2 (ROW)
- new net: D2.2 (A), MX2.2 (ROW)
- new net: D1.2 (A), MX1.2 (ROW)
- new net: D3.2 (A), MX3.2 (ROW)
- new net COL0: MX1.1 (COL), MX3.1 (COL)
- new net COL1: MX2.1 (COL), MX4.1 (COL)
- new net ROW0: D1.1 (K), D2.1 (K)
- new net ROW1: D3.1 (K), D4.1 (K)
- new net VCC: F1.1, USB1.6 (SHIELD)
