File: _autosave-bigMacro.kicad_pcb (KiCad board)
At the start: 2 copper layers, 85.7 x 38.1 mm, 25 parts, among them SW1 SW_Push, U1 ATmega32U4-A, Y1 16MHz

Commit message: Update Journal.MD
Parts:
- moved G*** 31.1 mm to (106.4, 101.6)
Changed lines of the file:
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@@
 	(footprint "LOGO"
 		(layer "B.Cu")
-		(at 135.651948 91.152804 180)
+		(at 106.3625 101.6 180)
 		(property "Reference" "G***"
 			(at 0 0 0)
@@
 	)
 	(gr_text "crappy wiring (c)\npart of this complete breakfast"
-		(at 141.2875 100.0125 0)
+		(at 111.91875 94.45625 0)
 		(layer "B.SilkS")
 		(effects
