File: bigMacro.kicad_pcb (KiCad board)
At the start: 2 copper layers, 100 x 76.3 mm, 36 parts, among them U2 XIAO-RP2040-DIP

Commit message: a
Parts:
- removed D9: D_Small, Diode_SMD:D_SOD-123
- removed MX7: MX-NoLED, Button_Switch_Keyboard:SW_Cherry_MX_1.00u_PCB
Routing:
- net /COL3: track 73.7 -> 54.6 mm
- net Net-(D9-A): track 15.6 -> 0.00 mm
