File: PCB/bigMacro.kicad_pcb (KiCad board)
At the start: 2 copper layers, 100 x 76.3 mm, 34 parts, among them U2 XIAO-RP2040-DIP

Commit message: PCB Design update
Parts:
- added D9: D_Small, Diode_SMD:D_SOD-123, F.Cu at (2.42, 16.3)
- added MX7: MX-NoLED, Button_Switch_Keyboard:SW_Cherry_MX_1.00u_PCB, F.Cu at (9.59, 1.97)
Connections:
- D5 pad 2: Net-(D5-VSS) -> GND
- D5 pad 4: Net-(D5-VDD) -> +5V
- D6 pad 2: Net-(D5-VSS) -> GND
- D6 pad 4: Net-(D5-VDD) -> +5V
Routing:
- net GND: track 0.00 -> 48.2 mm
- net +5V: track 0.00 -> 36.4 mm, vias 0 -> 1
- net Net-(D5-VSS): track 9.79 -> 0.00 mm
- net Net-(D5-VDD): track 9.66 -> 0.00 mm

Commit message: Redid PCB
Parts:
- removed D9: D_Small, Diode_SMD:D_SOD-123
- removed MX7: MX-NoLED, Button_Switch_Keyboard:SW_Cherry_MX_1.00u_PCB
